Commit message: added dreamwalker_dummy urdf

File: dreamwalker_description/urdf/dreamwalker_dummy.urdf (robot description, URDF)
Before this commit: robot dreamwalker, 17 links, 16 joints
Links:
- added link support_element, mass 0.8; collision box size=0.1 0.14 0.19; visual mesh filename=package://dreamwalker_description/meshes/support_test_eleme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 scale=0.001 0.001 0.001
Joints:
- added joint dummy_joint: type fixed, parent support_element, child main_body, origin xyz=0 0 0.19 rpy=0 0 0

Commit message: further URDF tweaks, added control package

File: dreamwalker_description/urdf/dreamwalker_dummy.urdf (robot description, URDF)
Before this commit: robot dreamwalker_dummy, 18 links, 17 joints
Links:
- link link_femur1: geometry collision box size=0.014 0.02 0.085; visual mesh filename=package://dreamwalker_description/meshes/link_femur1.stl scale=0.001 0.001 0.001
- link link_femur2: geometry collision box size=0.014 0.02 0.085; visual mesh filename=package://dreamwalker_description/meshes/link_femur2.stl scale=0.001 0.001 0.001
- link link_femur3: geometry collision box size=0.014 0.02 0.085; visual mesh filename=package://dreamwalker_description/meshes/link_femur3.stl scale=0.001 0.001 0.001
- link link_femur4: geometry collision box size=0.014 0.02 0.085; visual mesh filename=package://dreamwalker_description/meshes/link_femur4.stl scale=0.001 0.001 0.001
- link link_shoulder1: geometry collision box size=0.034 0.045 0.0175; visual mesh filename=package://dreamwalker_description/meshes/link_shoulder1.stl scale=0.001 0.001 0.001
- link link_shoulder2: geometry collision box size=0.034 0.045 0.0175; visual mesh filename=package://dreamwalker_description/meshes/link_shoulder2.stl scale=0.001 0.001 0.001
- link link_shoulder3: geometry collision box size=0.034 0.045 0.0175; visual mesh filename=package://dreamwalker_description/meshes/link_shoulder3.stl scale=0.001 0.001 0.001
- link link_shoulder4: geometry collision box size=0.034 0.045 0.0175; visual mesh filename=package://dreamwalker_description/meshes/link_shoulder4.stl scale=0.001 0.001 0.001
- link link_tibia1: geometry collision box size=0.005 0.015 0.075; visual mesh filename=package://dreamwalker_description/meshes/link_tibia1.stl scale=0.001 0.001 0.001
- link link_tibia2: geometry collision box size=0.005 0.015 0.075; visual mesh filename=package://dreamwalker_description/meshes/link_tibia2.stl scale=0.001 0.001 0.001
- link link_tibia3: geometry collision box size=0.005 0.015 0.075; visual mesh filename=package://dreamwalker_description/meshes/link_tibia3.stl scale=0.001 0.001 0.001
- link link_tibia4: geometry collision box size=0.005 0.015 0.075; visual mesh filename=package://dreamwalker_description/meshes/link_tibia4.stl scale=0.001 0.001 0.001
