Commit message: robot description urdf file modified

File: dreamwalker_description/urdf/dreamwalker.urdf (robot description, URDF)
Before this commit: robot dreamwalker, 1 links, 0 joints
Links:
- removed link link_base
- added link link_shoulder1, mass 0.0198; collision mesh filename=package://dreamwalker_description/meshes/link_shoulder1.stl scale=0.001 0.001 0.001; visual mesh filename=package://dreamwalker_description/meshes/link_shoulder1.stl scale=0.001 0.001 0.001
- added link link_shoulder2, mass 0.0198; collision mesh filename=package://dreamwalker_description/meshes/link_shoulder2.stl scale=0.001 0.001 0.001; visual mesh filename=package://dreamwalker_description/meshes/link_shoulder2.stl scale=0.001 0.001 0.001
- added link link_shoulder3, mass 0.0198; collision mesh filename=package://dreamwalker_description/meshes/link_shoulder3.stl scale=0.001 0.001 0.001; visual mesh filename=package://dreamwalker_description/meshes/link_shoulder3.stl scale=0.001 0.001 0.001
- added link link_shoulder4, mass 0.0198; collision mesh filename=package://dreamwalker_description/meshes/link_shoulder4.stl scale=0.001 0.001 0.001; visual mesh filename=package://dreamwalker_description/meshes/link_shoulder4.stl scale=0.001 0.001 0.001
- added link main_body, mass 0.388; collision mesh filename=package://dreamwalker_description/meshes/main_body_collisio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 scale=0.001 0.001 0.001; visual mesh filename=package://dreamwalker_description/meshes/main_body.stl scale=0.001 0.001 0.001
Joints:
- added joint shoulder_joint1: type continuous, parent main_body, child link_shoulder1, origin xyz=-0.062 0.064 0.022 rpy=0 0 0, axis 0 1 0
- added joint shoulder_joint2: type continuous, parent main_body, child link_shoulder2, origin xyz=0.062 0.064 0.022 rpy=0 0 0, axis 0 1 0
- added joint shoulder_joint3: type continuous, parent main_body, child link_shoulder3, origin xyz=-0.062 -0.064 0.022 rpy=0 0 0, axis 0 1 0
- added joint shoulder_joint4: type continuous, parent main_body, child link_shoulder4, origin xyz=0.062 -0.064 0.022 rpy=0 0 0, axis 0 1 0

Commit message: updated dreamwalker.urdf file

File: dreamwalker_description/urdf/dreamwalker.urdf (robot description, URDF)
Before this commit: robot dreamwalker, 5 links, 4 joints
Links:
- added link link_femur1, mass 0.0218; collision mesh filename=package://dreamwalker_description/meshes/link_femur1.stl scale=0.001 0.001 0.001; visual mesh filename=package://dreamwalker_description/meshes/link_femur1.stl scale=0.001 0.001 0.001
- added link link_femur2, mass 0.0218; collision mesh filename=package://dreamwalker_description/meshes/link_femur2.stl scale=0.001 0.001 0.001; visual mesh filename=package://dreamwalker_description/meshes/link_femur2.stl scale=0.001 0.001 0.001
- added link link_femur3, mass 0.0218; collision mesh filename=package://dreamwalker_description/meshes/link_femur3.stl scale=0.001 0.001 0.001; visual mesh filename=package://dreamwalker_description/meshes/link_femur3.stl scale=0.001 0.001 0.001
- added link link_femur4, mass 0.0218; collision mesh filename=package://dreamwalker_description/meshes/link_femur4.stl scale=0.001 0.001 0.001; visual mesh filename=package://dreamwalker_description/meshes/link_femur4.stl scale=0.001 0.001 0.001
- added link link_tibia1, mass 0.00651; collision mesh filename=package://dreamwalker_description/meshes/link_tibia1.stl scale=0.001 0.001 0.001; visual mesh filename=package://dreamwalker_description/meshes/link_tibia1.stl scale=0.001 0.001 0.001
- added link link_tibia2, mass 0.00651; collision mesh filename=package://dreamwalker_description/meshes/link_tibia2.stl scale=0.001 0.001 0.001; visual mesh filename=package://dreamwalker_description/meshes/link_tibia2.stl scale=0.001 0.001 0.001
- added link link_tibia3, mass 0.00651; collision mesh filename=package://dreamwalker_description/meshes/link_tibia3.stl scale=0.001 0.001 0.001; visual mesh filename=package://dreamwalker_description/meshes/link_tibia3.stl scale=0.001 0.001 0.001
- added link link_tibia4, mass 0.00651; collision mesh filename=package://dreamwalker_description/meshes/link_tibia4.stl scale=0.001 0.001 0.001; visual mesh filename=package://dreamwalker_description/meshes/link_tibia4.stl scale=0.001 0.001 0.001
Joints:
- added joint knee_joint1: type continuous, parent link_femur1, child link_tibia1, origin xyz=0.005 0 -0.055 rpy=0 0 0, axis 1 0 0
- added joint knee_joint2: type continuous, parent link_femur2, child link_tibia2, origin xyz=-0.005 0 -0.055 rpy=0 0 0, axis 1 0 0
- added joint knee_joint3: type continuous, parent link_femur3, child link_tibia3, origin xyz=0.005 0 -0.055 rpy=0 0 0, axis 1 0 0
- added joint knee_joint4: type continuous, parent link_femur4, child link_tibia4, origin xyz=-0.005 0 -0.055 rpy=0 0 0, axis 1 0 0
- added joint limb_joint1: type continuous, parent link_shoulder1, child link_femur1, origin xyz=-0.024 0.0305 0 rpy=0 0 0, axis 1 0 0
- added joint limb_joint2: type continuous, parent link_shoulder2, child link_femur2, origin xyz=0.024 0.0305 0 rpy=0 0 0, axis 1 0 0
- added joint limb_joint3: type continuous, parent link_shoulder3, child link_femur3, origin xyz=-0.024 -0.0305 0 rpy=0 0 0, axis 1 0 0
- added joint limb_joint4: type continuous, parent link_shoulder4, child link_femur4, origin xyz=0.024 -0.0305 0 rpy=0 0 0, axis 1 0 0

Commit message: new worlds added, some robot description parameters changed

File: dreamwalker_description/urdf/dreamwalker.urdf (robot description, URDF)
Before this commit: robot dreamwalker, 17 links, 16 joints
Links:
- link link_femur1: geometry collision box size=0.01 0.01 0.01; visual mesh filename=package://dreamwalker_description/meshes/link_femur1.stl scale=0.001 0.001 0.001
- link link_femur2: geometry collision box size=0.01 0.01 0.01; visual mesh filename=package://dreamwalker_description/meshes/link_femur2.stl scale=0.001 0.001 0.001
- link link_femur3: geometry collision box size=0.01 0.01 0.01; visual mesh filename=package://dreamwalker_description/meshes/link_femur3.stl scale=0.001 0.001 0.001
- link link_femur4: geometry collision box size=0.01 0.01 0.01; visual mesh filename=package://dreamwalker_description/meshes/link_femur4.stl scale=0.001 0.001 0.001
- link link_shoulder1: geometry collision box size=0.01 0.01 0.01; visual mesh filename=package://dreamwalker_description/meshes/link_shoulder1.stl scale=0.001 0.001 0.001
- link link_shoulder2: geometry collision box size=0.01 0.01 0.01; visual mesh filename=package://dreamwalker_description/meshes/link_shoulder2.stl scale=0.001 0.001 0.001
- link link_shoulder3: geometry collision box size=0.01 0.01 0.01; visual mesh filename=package://dreamwalker_description/meshes/link_shoulder3.stl scale=0.001 0.001 0.001
- link link_shoulder4: geometry collision box size=0.01 0.01 0.01; visual mesh filename=package://dreamwalker_description/meshes/link_shoulder4.stl scale=0.001 0.001 0.001
- link link_tibia1: geometry collision box size=0.01 0.01 0.01; visual mesh filename=package://dreamwalker_description/meshes/link_tibia1.stl scale=0.001 0.001 0.001
- link link_tibia2: geometry collision box size=0.01 0.01 0.01; visual mesh filename=package://dreamwalker_description/meshes/link_tibia2.stl scale=0.001 0.001 0.001
- link link_tibia3: geometry collision box size=0.01 0.01 0.01; visual mesh filename=package://dreamwalker_description/meshes/link_tibia3.stl scale=0.001 0.001 0.001
- link link_tibia4: geometry collision box size=0.01 0.01 0.01; visual mesh filename=package://dreamwalker_description/meshes/link_tibia4.stl scale=0.001 0.001 0.001

File: dreamwalker_description/urdf/dreamwalker_dummy.urdf (robot description, URDF)
Before this commit: robot dreamwalker_dummy, 18 links, 17 joints
Links:
- link link_femur1: geometry collision box size=0.01 0.01 0.01; visual mesh filename=package://dreamwalker_description/meshes/link_femur1.stl scale=0.001 0.001 0.001
- link link_femur2: geometry collision box size=0.01 0.01 0.01; visual mesh filename=package://dreamwalker_description/meshes/link_femur2.stl scale=0.001 0.001 0.001
- link link_femur3: geometry collision box size=0.01 0.01 0.01; visual mesh filename=package://dreamwalker_description/meshes/link_femur3.stl scale=0.001 0.001 0.001
- link link_femur4: geometry collision box size=0.01 0.01 0.01; visual mesh filename=package://dreamwalker_description/meshes/link_femur4.stl scale=0.001 0.001 0.001
- link link_shoulder1: geometry collision box size=0.1 0.01 0.01; visual mesh filename=package://dreamwalker_description/meshes/link_shoulder1.stl scale=0.001 0.001 0.001
- link link_shoulder2: geometry collision box size=0.01 0.01 0.01; visual mesh filename=package://dreamwalker_description/meshes/link_shoulder2.stl scale=0.001 0.001 0.001
- link link_shoulder3: geometry collision box size=0.01 0.01 0.01; visual mesh filename=package://dreamwalker_description/meshes/link_shoulder3.stl scale=0.001 0.001 0.001
- link link_shoulder4: geometry collision box size=0.01 0.01 0.01; visual mesh filename=package://dreamwalker_description/meshes/link_shoulder4.stl scale=0.001 0.001 0.001
- link link_tibia1: geometry collision box size=0.01 0.01 0.01; visual mesh filename=package://dreamwalker_description/meshes/link_tibia1.stl scale=0.001 0.001 0.001
- link link_tibia2: geometry collision box size=0.01 0.01 0.01; visual mesh filename=package://dreamwalker_description/meshes/link_tibia2.stl scale=0.001 0.001 0.001
- link link_tibia3: geometry collision box size=0.01 0.01 0.01; visual mesh filename=package://dreamwalker_description/meshes/link_tibia3.stl scale=0.001 0.001 0.001
- link link_tibia4: geometry collision box size=0.01 0.01 0.01; visual mesh filename=package://dreamwalker_description/meshes/link_tibia4.stl scale=0.001 0.001 0.001
- link support_element: geometry collision box size=0.06 0.14 0.19; visual mesh filename=package://dreamwalker_description/meshes/support_test_eleme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 scale=0.001 0.001 0.001
Joints:
- joint shoulder_joint1: limit lower=-0.5235987755983 upper=0.5235987755983 effort=30 velocity=1.0 -> lower=-0.5235987755983 upper=0.5235987755983 effort=30 velocity=5.0
- joint shoulder_joint2: limit lower=-0.5235987755983 upper=0.5235987755983 effort=30 velocity=1.0 -> lower=-0.5235987755983 upper=0.5235987755983 effort=30 velocity=5.0
- joint shoulder_joint3: limit lower=-0.5235987755983 upper=0.5235987755983 effort=30 velocity=1.0 -> lower=-0.5235987755983 upper=0.5235987755983 effort=30 velocity=5.0
- joint shoulder_joint4: limit lower=-0.5235987755983 upper=0.5235987755983 effort=30 velocity=1.0 -> lower=-0.52359 upper=0.52359 effort=30 velocity=1.0

Commit message: links collision models modified

File: dreamwalker_description/urdf/dreamwalker.urdf (robot description, URDF)
Before this commit: robot dreamwalker, 17 links, 16 joints
Links:
- link link_femur1: geometry collision box size=0.014 0.02 0.085; visual mesh filename=package://dreamwalker_description/meshes/link_femur1.stl scale=0.001 0.001 0.001
- link link_femur2: geometry collision box size=0.014 0.02 0.085; visual mesh filename=package://dreamwalker_description/meshes/link_femur2.stl scale=0.001 0.001 0.001
- link link_femur3: geometry collision box size=0.014 0.02 0.085; visual mesh filename=package://dreamwalker_description/meshes/link_femur3.stl scale=0.001 0.001 0.001
- link link_femur4: geometry collision box size=0.014 0.02 0.085; visual mesh filename=package://dreamwalker_description/meshes/link_femur4.stl scale=0.001 0.001 0.001
- link link_shoulder1: geometry collision box size=0.034 0.045 0.0175; visual mesh filename=package://dreamwalker_description/meshes/link_shoulder1.stl scale=0.001 0.001 0.001
- link link_shoulder2: geometry collision box size=0.034 0.045 0.0175; visual mesh filename=package://dreamwalker_description/meshes/link_shoulder2.stl scale=0.001 0.001 0.001
- link link_shoulder3: geometry collision box size=0.034 0.045 0.0175; visual mesh filename=package://dreamwalker_description/meshes/link_shoulder3.stl scale=0.001 0.001 0.001
- link link_shoulder4: geometry collision box size=0.034 0.045 0.0175; visual mesh filename=package://dreamwalker_description/meshes/link_shoulder4.stl scale=0.001 0.001 0.001
- link link_tibia1: geometry collision box size=0.005 0.015 0.075; visual mesh filename=package://dreamwalker_description/meshes/link_tibia1.stl scale=0.001 0.001 0.001
- link link_tibia2: geometry collision box size=0.005 0.015 0.075; visual mesh filename=package://dreamwalker_description/meshes/link_tibia2.stl scale=0.001 0.001 0.001
- link link_tibia3: geometry collision box size=0.005 0.015 0.075; visual mesh filename=package://dreamwalker_description/meshes/link_tibia3.stl scale=0.001 0.001 0.001
- link link_tibia4: geometry collision box size=0.005 0.015 0.075; visual mesh filename=package://dreamwalker_description/meshes/link_tibia4.stl scale=0.001 0.001 0.001
Joints:
- joint foot_joint1: origin xyz=-0.0025 0 -0.065 rpy=-0.5235987755983 0 0 -> xyz=-0.0025 0 -0.065 rpy=-0.52359 0 0
- joint foot_joint2: origin xyz=0.0025 0 -0.065 rpy=-0.5235987755983 0 0 -> xyz=0.0025 0 -0.065 rpy=-0.52359 0 0
- joint foot_joint3: origin xyz=-0.0025 0 -0.065 rpy=0.5235987755983 0 0 -> xyz=-0.0025 0 -0.065 rpy=0.52359 0 0
- joint foot_joint4: origin xyz=0.0025 0 -0.065 rpy=0.5235987755983 0 0 -> xyz=0.0025 0 -0.065 rpy=0.52359 0 0
- joint shoulder_joint1: limit lower=-0.5235987755983 upper=0.5235987755983 effort=30 velocity=1.0 -> lower=-0.5235987755983 upper=0.5235987755983 effort=30 velocity=5.0
- joint shoulder_joint2: limit lower=-0.5235987755983 upper=0.5235987755983 effort=30 velocity=1.0 -> lower=-0.5235987755983 upper=0.5235987755983 effort=30 velocity=5.0
- joint shoulder_joint3: limit lower=-0.5235987755983 upper=0.5235987755983 effort=30 velocity=1.0 -> lower=-0.5235987755983 upper=0.5235987755983 effort=30 velocity=5.0
- joint shoulder_joint4: limit lower=-0.5235987755983 upper=0.5235987755983 effort=30 velocity=1.0 -> lower=-0.52359 upper=0.52359 effort=30 velocity=1.0

File: dreamwalker_description/urdf/dreamwalker_dummy.urdf (robot description, URDF)
Before this commit: robot dreamwalker_dummy, 18 links, 17 joints
Joints:
- joint foot_joint1: origin xyz=-0.0025 0 -0.065 rpy=-0.5235987755983 0 0 -> xyz=-0.0025 0 -0.065 rpy=-0.52359 0 0
- joint foot_joint2: origin xyz=0.0025 0 -0.065 rpy=-0.5235987755983 0 0 -> xyz=0.0025 0 -0.065 rpy=-0.52359 0 0
- joint foot_joint3: origin xyz=-0.0025 0 -0.065 rpy=0.5235987755983 0 0 -> xyz=-0.0025 0 -0.065 rpy=0.52359 0 0
- joint foot_joint4: origin xyz=0.0025 0 -0.065 rpy=0.5235987755983 0 0 -> xyz=0.0025 0 -0.065 rpy=0.52359 0 0

Commit message: New DAE files added, fixed launch and urdf files, added control test files

File: dreamwalker_description/urdf/dreamwalker.urdf (robot description, URDF)
Before this commit: robot dreamwalker, 17 links, 16 joints
Links:
- added link dummy
Joints:
- added joint dummy_joint: type fixed, parent dummy, child main_body

File: dreamwalker_description/urdf/dreamwalker_dummy.urdf (robot description, URDF)
Before this commit: robot dreamwalker_dummy, 18 links, 17 joints
Links:
- added link world
- link link_foot1: geometry collision mesh filename=package://dreamwalker_description/meshes/link_foot.dae scale=0.001 0.001 0.001; visual mesh filename=package://dreamwalker_description/meshes/link_foot.dae scale=0.001 0.001 0.001
- link link_foot2: geometry collision mesh filename=package://dreamwalker_description/meshes/link_foot.dae scale=0.001 0.001 0.001; visual mesh filename=package://dreamwalker_description/meshes/link_foot.dae scale=0.001 0.001 0.001
- link link_foot3: geometry collision mesh filename=package://dreamwalker_description/meshes/link_foot.dae scale=0.001 0.001 0.001; visual mesh filename=package://dreamwalker_description/meshes/link_foot.dae scale=0.001 0.001 0.001
- link link_foot4: geometry collision mesh filename=package://dreamwalker_description/meshes/link_foot.dae scale=0.001 0.001 0.001; visual mesh filename=package://dreamwalker_description/meshes/link_foot.dae scale=0.001 0.001 0.001
- link link_tibia1: geometry collision box size=0.005 0.015 0.075; visual mesh filename=package://dreamwalker_description/meshes/link_tibia1.dae scale=0.001 0.001 0.001
Joints:
- added joint fixed: type fixed, parent world, child support_element

Commit message: some precious control files added

File: dreamwalker_description/urdf/dreamwalker.urdf (robot description, URDF)
Before this commit: robot dreamwalker, 22 links, 21 joints
Links:
- removed link world
- link link_foot1: geometry collision mesh filename=package://dreamwalker_description/meshes/link_foot.stl scale=0.001 0.001 0.001; visual mesh filename=package://dreamwalker_description/meshes/link_foot.stl scale=0.001 0.001 0.001
- link link_foot2: geometry collision mesh filename=package://dreamwalker_description/meshes/link_foot.stl scale=0.001 0.001 0.001; visual mesh filename=package://dreamwalker_description/meshes/link_foot.stl scale=0.001 0.001 0.001
- link link_foot3: geometry collision mesh filename=package://dreamwalker_description/meshes/link_foot.stl scale=0.001 0.001 0.001; visual mesh filename=package://dreamwalker_description/meshes/link_foot.stl scale=0.001 0.001 0.001
- link link_foot4: geometry collision mesh filename=package://dreamwalker_description/meshes/link_foot.stl scale=0.001 0.001 0.001; visual mesh filename=package://dreamwalker_description/meshes/link_foot.stl scale=0.001 0.001 0.001
Joints:
- removed joint world_joint
- joint b_sensor_joint: limit lower=0 upper=0 effort=1000 velocity=0.0 -> (none); type revolute -> fixed
- joint l_sensor_joint: limit lower=0 upper=0 effort=1000 velocity=0.0 -> (none); type revolute -> fixed
- joint m_sensor_joint: limit lower=0 upper=0 effort=1000 velocity=0.0 -> (none); type revolute -> fixed
- joint r_sensor_joint: limit lower=0 upper=0 effort=1000 velocity=0.0 -> (none); type revolute -> fixed
- joint shoulder_joint1: limit lower=-0.5235987755983 upper=0.5235987755983 effort=2.5 velocity=1.0 -> lower=-0.5235987755983 upper=0.5235987755983 effort=30 velocity=5.0
- joint shoulder_joint2: limit lower=-0.5235987755983 upper=0.5235987755983 effort=2.5 velocity=5.0 -> lower=-0.5235987755983 upper=0.5235987755983 effort=30 velocity=5.0
- joint shoulder_joint3: limit lower=-0.5235987755983 upper=0.5235987755983 effort=2.5 velocity=5.0 -> lower=-0.5235987755983 upper=0.5235987755983 effort=30 velocity=5.0
- joint shoulder_joint4: limit lower=-0.52359 upper=0.52359 effort=2.5 velocity=1.0 -> lower=-0.52359 upper=0.52359 effort=30 velocity=1.0

File: dreamwalker_description/urdf/dreamwalker_dummy.urdf (robot description, URDF)
Before this commit: robot dreamwalker, 22 links, 21 joints
Links:
- added link support_element, mass 0.8; collision box size=0.06 0.14 0.19; visual mesh filename=package://dreamwalker_description/meshes/support_test_eleme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 scale=0.001 0.001 0.001
- link link_foot1: geometry collision mesh filename=package://dreamwalker_description/meshes/link_foot.dae scale=0.001 0.001 0.001; visual mesh filename=package://dreamwalker_description/meshes/link_foot.dae scale=0.001 0.001 0.001
- link link_foot2: geometry collision mesh filename=package://dreamwalker_description/meshes/link_foot.dae scale=0.001 0.001 0.001; visual mesh filename=package://dreamwalker_description/meshes/link_foot.dae scale=0.001 0.001 0.001
- link link_foot3: geometry collision mesh filename=package://dreamwalker_description/meshes/link_foot.dae scale=0.001 0.001 0.001; visual mesh filename=package://dreamwalker_description/meshes/link_foot.dae scale=0.001 0.001 0.001
- link link_foot4: geometry collision mesh filename=package://dreamwalker_description/meshes/link_foot.dae scale=0.001 0.001 0.001; visual mesh filename=package://dreamwalker_description/meshes/link_foot.dae scale=0.001 0.001 0.001
Joints:
- removed joint world_joint
- added joint dummy_joint: type fixed, parent support_element, child main_body, origin xyz=0 0 0.19 rpy=0 0 0
- added joint fixed: type fixed, parent world, child support_element
- joint b_sensor_joint: limit lower=0 upper=0 effort=1000 velocity=0.0 -> (none); type revolute -> fixed
- joint l_sensor_joint: limit lower=0 upper=0 effort=1000 velocity=0.0 -> (none); type revolute -> fixed
- joint m_sensor_joint: limit lower=0 upper=0 effort=1000 velocity=0.0 -> (none); type revolute -> fixed
- joint r_sensor_joint: limit lower=0 upper=0 effort=1000 velocity=0.0 -> (none); type revolute -> fixed
- joint shoulder_joint1: limit lower=-0.5235987755983 upper=0.5235987755983 effort=2.5 velocity=1.0 -> lower=-0.5235987755983 upper=0.5235987755983 effort=30 velocity=5.0
- joint shoulder_joint2: limit lower=-0.5235987755983 upper=0.5235987755983 effort=2.5 velocity=5.0 -> lower=-0.5235987755983 upper=0.5235987755983 effort=30 velocity=5.0
- joint shoulder_joint3: limit lower=-0.5235987755983 upper=0.5235987755983 effort=2.5 velocity=5.0 -> lower=-0.5235987755983 upper=0.5235987755983 effort=30 velocity=5.0
- joint shoulder_joint4: limit lower=-0.52359 upper=0.52359 effort=2.5 velocity=1.0 -> lower=-0.52359 upper=0.52359 effort=30 velocity=1.0
