Commit message: kinda able to walk

File: dreamwalker_description/urdf/dreamwalker_test.xacro (robot description, xacro)
@@ -39,5 +39,5 @@
 			<inertia ixx="0.000003218011" ixy="0.000000199995" ixz="0" iyy="0.000001946476" iyz="0" izz="0.000004027678"/>
 		</inertial>
-		<collision>
+		<collision name="collision_base">
 			<origin xyz="-0.007 0.0225 0" rpy="0 0 0"/>
 			<geometry>
@@ -77,5 +77,5 @@
 			<inertia ixx="0.000003218011" ixy="-0.000000199995" ixz="0" iyy="0.000001946476" iyz="0" izz="0.000004027678"/>
 		</inertial>
-		<collision>
+		<collision name="collision_base">
 			<origin xyz="-0.007 -0.0225 0" rpy="0 0 0"/>
 			<geometry>
@@ -96,5 +96,5 @@
 			<inertia ixx="0.000003218011" ixy="0.000000199995" ixz="0" iyy="0.000001946476" iyz="0" izz="0.000004027678"/>
 		</inertial>
-		<collision>
+		<collision name="collision_base">
 			<origin xyz="0.007 -0.0225 0" rpy="0 0 0"/>
 			<geometry>
@@ -127,5 +127,5 @@
 				<mesh filename="package://dreamwalker_description/meshes/link_femur1.stl" scale="0.001 0.001 0.001" />
 			</geometry>
-			<material name="red"/>
+			<material name="black"/>
 		</visual>
 	</link>
@@ -147,5 +147,5 @@
 				<mesh filename="package://dreamwalker_description/meshes/link_femur2.stl" scale="0.001 0.001 0.001" />
 			</geometry>
-			<material name="red"/>
+			<material name="black"/>
 		</visual>
 	</link>
@@ -167,5 +167,5 @@
 				<mesh filename="package://dreamwalker_description/meshes/link_femur3.stl" scale="0.001 0.001 0.001" />
 			</geometry>
-			<material name="red"/>
+			<material name="black"/>
 		</visual>
 	</link>
@@ -187,5 +187,5 @@
 				<mesh filename="package://dreamwalker_description/meshes/link_femur4.stl" scale="0.001 0.001 0.001" />
 			</geometry>
-			<material name="red"/>
+			<material name="black"/>
 		</visual>
 	</link>
@@ -275,5 +275,5 @@
 			<origin xyz="0 0 0" rpy="0 0 0"/>
 			<geometry>
-				<mesh filename="package://dreamwalker_description/meshes/link_foot.stl" scale="0.001 0.001 0.001" />
+				<mesh filename="package://dreamwalker_description/meshes/link_foot.dae" scale="0.001 0.001 0.001" />
 			</geometry>
 			<!-- <contact_coefficient mu="100.0" mu2="100.0" k_p="10000.0"  k_d="100.0" /> -->
@@ -296,5 +296,5 @@
 			<origin xyz="0 0 0" rpy="0 0 0"/>
 			<geometry>
-				<mesh filename="package://dreamwalker_description/meshes/link_foot.stl" scale="0.001 0.001 0.001" />
+				<mesh filename="package://dreamwalker_description/meshes/link_foot.dae" scale="0.001 0.001 0.001" />
 			</geometry>
 			<!-- <contact_coefficient mu="100.0" mu2="100.0" k_p="10000.0"  k_d="100.0" /> -->
@@ -317,5 +317,5 @@
 			<origin xyz="0 0 0" rpy="0 0 0"/>
 			<geometry>
-				<mesh filename="package://dreamwalker_description/meshes/link_foot.stl" scale="0.001 0.001 0.001" />
+				<mesh filename="package://dreamwalker_description/meshes/link_foot.dae" scale="0.001 0.001 0.001" />
 			</geometry>
 			<!-- <contact_coefficient mu="100.0" mu2="100.0" k_p="10000.0"  k_d="100.0" /> -->
@@ -338,5 +338,5 @@
 			<origin xyz="0 0 0" rpy="0 0 0"/>
 			<geometry>
-				<mesh filename="package://dreamwalker_description/meshes/link_foot.stl" scale="0.001 0.001 0.001" />
+				<mesh filename="package://dreamwalker_description/meshes/link_foot.dae" scale="0.001 0.001 0.001" />
 			</geometry>
 			<!-- <contact_coefficient mu="100.0" mu2="100.0" k_p="10000.0"  k_d="100.0" /> -->
@@ -357,4 +357,5 @@
 		<child link="link_shoulder1"/>
 		<limit effort="2.5" velocity="1.0" lower="-0.5235987755983" upper="0.5235987755983" />
+		<!-- <dynamics damping="0.0" friction="1.0"/> -->
 	</joint>
 	<joint name="shoulder_joint2" type="revolute">
@@ -363,5 +364,5 @@
 		<parent link="main_body"/>
 		<child link="link_shoulder2"/>
-		<limit effort="2.5" velocity="5.0" lower="-0.5235987755983" upper="0.5235987755983" />
+		<limit effort="2.5" velocity="1.0" lower="-0.5235987755983" upper="0.5235987755983" />
 		<!-- <dynamics damping="0.0" friction="1.0"/> -->
 	</joint>
@@ -371,5 +372,5 @@
 		<parent link="main_body"/>
 		<child link="link_shoulder3"/>
-		<limit effort="2.5" velocity="5.0" lower="-0.5235987755983" upper="0.5235987755983" />
+		<limit effort="2.5" velocity="1.0" lower="-0.5235987755983" upper="0.5235987755983" />
 		<!--<dynamics damping="0.0" friction="1.0"/> -->
 	</joint>
@@ -387,5 +388,5 @@
 		<parent link="link_shoulder1"/>
 		<child link="link_femur1"/>
-		<limit effort="30" velocity="1.0" lower="-1.57079" upper="1.57079" />
+		<limit effort="2.5" velocity="1.0" lower="-1.57079" upper="1.57079" />
 		<!-- <dynamics damping="0.0" friction="1.0"/> -->
 	</joint>
@@ -395,5 +396,5 @@
 		<parent link="link_shoulder2"/>
 		<child link="link_femur2"/>
-		<limit effort="30" velocity="1.0" lower="-1.57079" upper="1.57079" />
+		<limit effort="2.5" velocity="1.0" lower="-1.57079" upper="1.57079" />
 		<!-- <dynamics damping="0.0" friction="1.0"/> -->
 	</joint>
@@ -403,5 +404,5 @@
 		<parent link="link_shoulder3"/>
 		<child link="link_femur3"/>
-		<limit effort="30" velocity="1.0" lower="-1.57079" upper="1.57079" />
+		<limit effort="2.5" velocity="1.0" lower="-1.57079" upper="1.57079" />
 		<!-- <dynamics damping="0.0" friction="1.0"/> -->
 	</joint>
@@ -411,5 +412,5 @@
 		<parent link="link_shoulder4"/>
 		<child link="link_femur4"/>
-		<limit effort="30" velocity="1.0" lower="-1.57079" upper="1.57079" />
+		<limit effort="2.5" velocity="1.0" lower="-1.57079" upper="1.57079" />
 		<!-- <dynamics damping="0.0" friction="1.0"/> -->
 	</joint>
@@ -419,5 +420,5 @@
 		<parent link="link_femur1"/>
 		<child link="link_tibia1"/>
-		<limit effort="30" velocity="1.0" lower="0" upper="2.09439" />
+		<limit effort="2.5" velocity="1.0" lower="0" upper="2.09439" />
 		<!-- <dynamics damping="0.0" friction="1.0"/> -->
 	</joint>
@@ -427,5 +428,5 @@
 		<parent link="link_femur2"/>
 		<child link="link_tibia2"/>
-		<limit effort="30" velocity="1.0" lower="0" upper="2.09439" />
+		<limit effort="2.5" velocity="1.0" lower="0" upper="2.09439" />
 		<!-- <dynamics damping="0.0" friction="1.0"/> -->
 	</joint>
@@ -435,5 +436,5 @@
 		<parent link="link_femur3"/>
 		<child link="link_tibia3"/>
-		<limit effort="30" velocity="1.0" lower="0" upper="2.09439" />
+		<limit effort="2.5" velocity="1.0" lower="0" upper="2.09439" />
 		<!-- <dynamics damping="0.0" friction="1.0"/> -->
 	</joint>
@@ -443,5 +444,5 @@
 		<parent link="link_femur4"/>
 		<child link="link_tibia4"/>
-		<limit effort="30" velocity="1.0" lower="0" upper="2.09439" />
+		<limit effort="2.5" velocity="1.0" lower="0" upper="2.09439" />
 		<!-- <dynamics damping="0.0" friction="1.0"/> -->
 	</joint>
