Commit message: Switched .urdf to .xacro format. Added sensors and solved friction problem. Deleted unused files

File: dreamwalker_description/urdf/dreamwalker_dummy.xacro (robot description, xacro)
@@ -1,4 +1,6 @@
 <?xml version="1.0" ?>
 <robot name="dreamwalker_dummy" xmlns:xacro="http://www.ros.org/wiki/xacro">
+	<xacro:include filename="$(find dreamwalker_description)/urdf/dreamwalker.gazebo" />
+  	<xacro:include filename="$(find dreamwalker_description)/urdf/materials.xacro" />
 	<!-- WORLD LINK -->
 	<link name="world"/>
@@ -27,4 +29,10 @@
 		</visual>
 	</link>
+	<joint name="dummy_joint" type="revolute">
+		<origin xyz="0 0 0.19" rpy="0 0 0"/>
+		<parent link="support_element"/>
+		<child link="main_body"/>
+		<limit effort="1000" velocity="0.0" lower="0" upper="0" />
+	</joint>
 	<!--### ROBOT BODY ### -->
 	<link name="main_body">
@@ -210,18 +218,18 @@
 	<link name="link_tibia1">
 		<inertial>
-			<mass value="0.00651"/>
-			<origin xyz="-0.0025 0.000876 -0.027677" rpy="0 0 0"/>
-			<inertia ixx="0.000003593654" ixy="0" ixz="0" iyy="0.000003455444" iyz="0.000000074876" izz="0.000000165334"/>
-		</inertial>
-		<collision name="collision_base">
-			<origin xyz="-0.0025 0 -0.028" rpy="0 0 0"/>
-			<geometry>
-				<box size="0.005 0.015 0.075"/>
-			</geometry>
-		</collision>
-		<visual>
-			<origin xyz="0 0 0" rpy="0 0 0"/>
-			<geometry>
-				<mesh filename="package://dreamwalker_description/meshes/link_tibia1.dae" scale="0.001 0.001 0.001" />
+			<mass value="0.00730"/>
+			<origin xyz="-0.0025 0.0009 -0.032102" rpy="0 0 0"/>
+			<inertia ixx="0.0000050464" ixy="0" ixz="0" iyy="0.000004893134" iyz="0.00000009901" izz="0.00000018368"/>
+		</inertial>
+		<collision name="collision_base">
+			<origin xyz="-0.0025 0 -0.033" rpy="0 0 0"/>
+			<geometry>
+				<box size="0.005 0.015 0.085"/>
+			</geometry>
+		</collision>
+		<visual>
+			<origin xyz="0 0 0" rpy="0 0 0"/>
+			<geometry>
+				<mesh filename="package://dreamwalker_description/meshes/link_forearm1.stl" scale="0.001 0.001 0.001" />
 			</geometry>
 		</visual>
@@ -229,18 +237,18 @@
 	<link name="link_tibia2">
 		<inertial>
-			<mass value="0.00651"/>
-			<origin xyz="0.0025 0.000876 -0.027677" rpy="0 0 0"/>
-			<inertia ixx="0.000003593654" ixy="0" ixz="0" iyy="0.000003455444" iyz="0.000000074876" izz="0.000000165334"/>
-		</inertial>
-		<collision name="collision_base">
-			<origin xyz="0.0025 0 -0.028" rpy="0 0 0"/>
-			<geometry>
-				<box size="0.005 0.015 0.075"/>
-			</geometry>
-		</collision>
-		<visual>
-			<origin xyz="0 0 0" rpy="0 0 0"/>
-			<geometry>
-				<mesh filename="package://dreamwalker_description/meshes/link_tibia2.stl" scale="0.001 0.001 0.001" />
+			<mass value="0.00730"/>
+			<origin xyz="0.0025 0.0009 -0.032102" rpy="0 0 0"/>
+			<inertia ixx="0.0000050464" ixy="0" ixz="0" iyy="0.000004893134" iyz="0.00000009901" izz="0.00000018368"/>
+		</inertial>
+		<collision name="collision_base">
+			<origin xyz="0.0025 0 -0.033" rpy="0 0 0"/>
+			<geometry>
+				<box size="0.005 0.015 0.085"/>
+			</geometry>
+		</collision>
+		<visual>
+			<origin xyz="0 0 0" rpy="0 0 0"/>
+			<geometry>
+				<mesh filename="package://dreamwalker_description/meshes/link_forearm2.stl" scale="0.001 0.001 0.001" />
 			</geometry>
 		</visual>
@@ -248,18 +256,18 @@
 	<link name="link_tibia3">
 		<inertial>
-			<mass value="0.00651"/>
-			<origin xyz="-0.0025 -0.000876 -0.027677" rpy="0 0 0"/>
-			<inertia ixx="0.000003593654" ixy="0" ixz="0" iyy="0.000003455444" iyz="-0.000000074876" izz="0.000000165334"/>
-		</inertial>
-		<collision name="collision_base">
-			<origin xyz="-0.0025 0 -0.028" rpy="0 0 0"/>
-			<geometry>
-				<box size="0.005 0.015 0.075"/>
-			</geometry>
-		</collision>
-		<visual>
-			<origin xyz="0 0 0" rpy="0 0 0"/>
-			<geometry>
-				<mesh filename="package://dreamwalker_description/meshes/link_tibia3.stl" scale="0.001 0.001 0.001" />
+			<mass value="0.00730"/>
+			<origin xyz="-0.0025 0.0009 -0.032102" rpy="0 0 0"/>
+			<inertia ixx="0.0000050464" ixy="0" ixz="0" iyy="0.000004893134" iyz="0.00000009901" izz="0.00000018368"/>
+		</inertial>
+		<collision name="collision_base">
+			<origin xyz="-0.0025 0 -0.033" rpy="0 0 0"/>
+			<geometry>
+				<box size="0.005 0.015 0.085"/>
+			</geometry>
+		</collision>
+		<visual>
+			<origin xyz="0 0 0" rpy="0 0 0"/>
+			<geometry>
+				<mesh filename="package://dreamwalker_description/meshes/link_forearm1.stl" scale="0.001 0.001 0.001" />
 			</geometry>
 		</visual>
@@ -267,18 +275,18 @@
 	<link name="link_tibia4">
 		<inertial>
-			<mass value="0.00651"/>
-			<origin xyz="0.0025 -0.000876 -0.027677" rpy="0 0 0"/>
-			<inertia ixx="0.000003593654" ixy="0" ixz="0" iyy="0.000003455444" iyz="-0.000000074876" izz="0.000000165334"/>
-		</inertial>
-		<collision name="collision_base">
-			<origin xyz="0.0025 0 -0.028" rpy="0 0 0"/>
-			<geometry>
-				<box size="0.005 0.015 0.075"/>
-			</geometry>
-		</collision>
-		<visual>
-			<origin xyz="0 0 0" rpy="0 0 0"/>
-			<geometry>
-				<mesh filename="package://dreamwalker_description/meshes/link_tibia4.stl" scale="0.001 0.001 0.001" />
+			<mass value="0.00730"/>
+			<origin xyz="0.0025 0.0009 -0.032102" rpy="0 0 0"/>
+			<inertia ixx="0.0000050464" ixy="0" ixz="0" iyy="0.000004893134" iyz="0.00000009901" izz="0.00000018368"/>
+		</inertial>
+		<collision name="collision_base">
+			<origin xyz="0.0025 0 -0.033" rpy="0 0 0"/>
+			<geometry>
+				<box size="0.005 0.015 0.085"/>
+			</geometry>
+		</collision>
+		<visual>
+			<origin xyz="0 0 0" rpy="0 0 0"/>
+			<geometry>
+				<mesh filename="package://dreamwalker_description/meshes/link_forearm2.stl" scale="0.001 0.001 0.001" />
 			</geometry>
 		</visual>
@@ -290,5 +298,5 @@
 			<inertia ixx="0.000000043185" ixy="0" ixz="0" iyy="0.000000029326" iyz="-0.000000074876" izz="0.000000054089"/>
 		</inertial>
-		<collision name="collision_base">
+		<collision>
 			<origin xyz="0 0 0" rpy="0 0 0"/>
 			<geometry>
@@ -311,5 +319,5 @@
 			<inertia ixx="0.000000043185" ixy="0" ixz="0" iyy="0.000000029326" iyz="-0.000000074876" izz="0.000000054089"/>
 		</inertial>
-		<collision name="collision_base">
+		<collision>
 			<origin xyz="0 0 0" rpy="0 0 0"/>
 			<geometry>
@@ -332,5 +340,5 @@
 			<inertia ixx="0.000000043185" ixy="0" ixz="0" iyy="0.000000029326" iyz="-0.000000074876" izz="0.000000054089"/>
 		</inertial>
-		<collision name="collision_base">
+		<collision>
 			<origin xyz="0 0 0" rpy="0 0 0"/>
 			<geometry>
@@ -353,5 +361,5 @@
 			<inertia ixx="0.000000043185" ixy="0" ixz="0" iyy="0.000000029326" iyz="-0.000000074876" izz="0.000000054089"/>
 		</inertial>
-		<collision name="collision_base">
+		<collision>
 			<origin xyz="0 0 0" rpy="0 0 0"/>
 			<geometry>
@@ -369,9 +377,4 @@
 	</link>
 	<!-- ### JOINTS ### -->
-	<joint name="dummy_joint" type="fixed">
-		<origin xyz="0 0 0.19" rpy="0 0 0"/>
-		<parent link="support_element"/>
-		<child link="main_body"/>
-	</joint>
 	<joint name="shoulder_joint1" type="revolute">
 		<origin xyz="-0.062 0.064 0.022" rpy="0 0 0"/>
@@ -459,5 +462,5 @@
 		<parent link="link_femur3"/>
 		<child link="link_tibia3"/>
-		<limit effort="30" velocity="1.0" lower="-2.09439" upper="0" />
+		<limit effort="30" velocity="1.0" lower="0" upper="2.09439" />
 		<!-- <dynamics damping="0.0" friction="1.0"/> -->
 	</joint>
@@ -467,33 +470,128 @@
 		<parent link="link_femur4"/>
 		<child link="link_tibia4"/>
-		<limit effort="30" velocity="1.0" lower="-2.09439" upper="0" />
+		<limit effort="30" velocity="1.0" lower="0" upper="2.09439" />
 		<!-- <dynamics damping="0.0" friction="1.0"/> -->
 	</joint>
 	<joint name="foot_joint1" type="fixed">
-		<origin xyz="-0.0025 0 -0.065" rpy="-0.52359 0 0"/>
+		<origin xyz="-0.0025 0 -0.075" rpy="-0.52359 0 0"/>
 		<parent link="link_tibia1"/>
 		<child link="link_foot1"/>
 	</joint>
 	<joint name="foot_joint2" type="fixed">
-		<origin xyz="0.0025 0 -0.065" rpy="-0.52359 0 0"/>
+		<origin xyz="0.0025 0 -0.075" rpy="-0.52359 0 0"/>
 		<parent link="link_tibia2"/>
 		<child link="link_foot2"/>
 	</joint>
 	<joint name="foot_joint3" type="fixed">
-		<origin xyz="-0.0025 0 -0.065" rpy="0.52359 0 0"/>
+		<origin xyz="-0.0025 0 -0.075" rpy="-0.52359 0 0"/>
 		<parent link="link_tibia3"/>
 		<child link="link_foot3"/>
 	</joint>
 	<joint name="foot_joint4" type="fixed">
-		<origin xyz="0.0025 0 -0.065" rpy="0.52359 0 0"/>
+		<origin xyz="0.0025 0 -0.075" rpy="-0.52359 0 0"/>
 		<parent link="link_tibia4"/>
 		<child link="link_foot4"/>
 	</joint>
-	<!-- ### GAZEBO ### -->
-	<gazebo>
-  		<plugin name="gazebo_ros_control" filename="libgazebo_ros_control.so">
-    		<robotNamespace>/dreamwalker</robotNamespace>
-  		</plugin>
-	</gazebo>
+	<!-- ### SENSORS ### -->
+	<link name="link_m_sensor">
+		<inertial>
+			<mass value="0.0102"/>
+			<origin xyz="0 0.01591 0.011" rpy="0 0 0"/>
+			<inertia ixx="0.000000566328" ixy="0" ixz="0" iyy="0.000002259218" iyz="-0.0000000944" izz="0.000002156532"/>
+		</inertial>
+		<collision name="collision_base">
+			<origin xyz="0 0.015 0.01125" rpy="0 0 0"/>
+			<geometry>
+				<box size="0.050 0.0293 0.0225"/>
+			</geometry>
+		</collision>
+		<visual>
+			<origin xyz="0 0 0" rpy="0 0 0"/>
+			<geometry>
+				<mesh filename="package://dreamwalker_description/meshes/link_fb_sensor.stl" scale="0.001 0.001 0.001" />
+			</geometry>
+		</visual>
+	</link>
+	<joint name="m_sensor_joint" type="revolute">
+		<origin xyz="0 0.095 0.005" rpy="0 0 0"/>
+		<parent link="main_body"/>
+		<child link="link_m_sensor"/>
+		<limit effort="1000" velocity="0.0" lower="0" upper="0" />
+	</joint>
+	<link name="link_b_sensor">
+		<inertial>
+			<mass value="0.0102"/>
+			<origin xyz="0 0.01591 0.011" rpy="0 0 0"/>
+			<inertia ixx="0.000000566328" ixy="0" ixz="0" iyy="0.000002259218" iyz="-0.0000000944" izz="0.000002156532"/>
+		</inertial>
+		<collision name="collision_base">
+			<origin xyz="0 0.015 0.01125" rpy="0 0 0"/>
+			<geometry>
+				<box size="0.050 0.0293 0.0225"/>
+			</geometry>
+		</collision>
+		<visual>
+			<origin xyz="0 0 0" rpy="0 0 0"/>
+			<geometry>
+				<mesh filename="package://dreamwalker_description/meshes/link_fb_sensor.stl" scale="0.001 0.001 0.001" />
+			</geometry>
+		</visual>
+	</link>
+	<joint name="b_sensor_joint" type="revolute">
+		<origin xyz="0 -0.095 0.005" rpy="0 0 3.141592"/>
+		<parent link="main_body"/>
+		<child link="link_b_sensor"/>
+		<limit effort="1000" velocity="0.0" lower="0" upper="0" />
+	</joint>
+	<link name="link_l_sensor">
+		<inertial>
+			<mass value="0.00983"/>
+			<origin xyz="0 0.01336 0.02495" rpy="0 0 0"/>
+			<inertia ixx="0.000002392374" ixy="0" ixz="0" iyy="0.000002455416" iyz="-0.000000093261" izz="0.000000406513"/>
+		</inertial>
+		<collision name="collision_base">
+			<origin xyz="0 0.015 0.025" rpy="0 0 0"/>
+			<geometry>
+				<box size="0.020 0.015 0.052"/>
+			</geometry>
+		</collision>
+		<visual>
+			<origin xyz="0 0 0" rpy="0 0 0"/>
+			<geometry>
+				<mesh filename="package://dreamwalker_description/meshes/link_rl_sensor.stl" scale="0.001 0.001 0.001" />
+			</geometry>
+		</visual>
+	</link>
+	<joint name="l_sensor_joint" type="revolute">
+		<origin xyz="-0.025 0.090 0.034" rpy="0 0 0.785398163"/>
+		<parent link="main_body"/>
+		<child link="link_l_sensor"/>
+		<limit effort="1000" velocity="0.0" lower="0" upper="0" />
+	</joint>
+	<link name="link_r_sensor">
+		<inertial>
+			<mass value="0.00983"/>
+			<origin xyz="0 0.01336 0.02495" rpy="0 0 0"/>
+			<inertia ixx="0.000002392374" ixy="0" ixz="0" iyy="0.000002455416" iyz="-0.000000093261" izz="0.000000406513"/>
+		</inertial>
+		<collision name="collision_base">
+			<origin xyz="0 0.015 0.025" rpy="0 0 0"/>
+			<geometry>
+				<box size="0.020 0.015 0.052"/>
+			</geometry>
+		</collision>
+		<visual>
+			<origin xyz="0 0 0" rpy="0 0 0"/>
+			<geometry>
+				<mesh filename="package://dreamwalker_description/meshes/link_rl_sensor.stl" scale="0.001 0.001 0.001" />
+			</geometry>
+		</visual>
+	</link>
+	<joint name="r_sensor_joint" type="revolute">
+		<origin xyz="0.025 0.090 0.034" rpy="0 0 -0.785398163"/>
+		<parent link="main_body"/>
+		<child link="link_r_sensor"/>
+		<limit effort="1000" velocity="0.0" lower="0" upper="0" />
+	</joint>
 	<!-- ### TRANSMISSIONS -->
 	<transmission name="tran_sh1">
@@ -617,30 +715,3 @@
     	</actuator>
   	</transmission>
-	<!-- COLORS AND FRICTION PARAMETERS -->
-	<gazebo reference="main_body">
-    	<material>Gazebo/Grey</material>
-  	</gazebo>
-  	<gazebo reference="link_foot1">
-    	<!-- using sdf block syntax directly in extension -->
-    	<collision>
-      		<friction>
-        		<ode>
-          			<mu>1.5</mu>
-          			<mu2>1.5</mu2>
-        		</ode>
-      		</friction>
-    	</collision>
-  	</gazebo>
-  	<gazebo reference="link_foot1">
-    	<material>Gazebo/Black</material>
-  	</gazebo>
-  	<gazebo reference="link_foot2">
-    	<material>Gazebo/Black</material>
-  	</gazebo>
-  	<gazebo reference="link_foot3">
-    	<material>Gazebo/Black</material>
-  	</gazebo>
-  	<gazebo reference="link_foot4">
-    	<material>Gazebo/Black</material>
-  	</gazebo>
 </robot>
