Commit message: Switched .urdf to .xacro format. Added sensors and solved friction problem. Deleted unused files

File: dreamwalker_description/urdf/dreamwalker_test.xacro (robot description, xacro)
@@ -1,12 +1,13 @@
 <?xml version="1.0" ?>
 <robot name="dreamwalker" xmlns:xacro="http://www.ros.org/wiki/xacro">
-	<!-- DUMMY LINK -->
-	<link name="dummy">
-	</link>
-	<joint name="dummy_joint" type="fixed">
-    	<parent link="dummy"/>
+	<xacro:include filename="$(find dreamwalker_description)/urdf/dreamwalker.gazebo" />
+  	<xacro:include filename="$(find dreamwalker_description)/urdf/materials.xacro" />
+	<!-- WORLD LINK -->
+	<link name="world"/>
+  	<joint name="world_joint" type="floating">
+    	<parent link="world"/>
     	<child link="main_body"/>
-    </joint>
-	<!--### BODY ### -->
+  	</joint>
+	<!--### ROBOT BODY ### -->
 	<link name="main_body">
 		<inertial>
@@ -191,18 +192,18 @@
 	<link name="link_tibia1">
 		<inertial>
-			<mass value="0.00651"/>
-			<origin xyz="-0.0025 0.000876 -0.027677" rpy="0 0 0"/>
-			<inertia ixx="0.000003593654" ixy="0" ixz="0" iyy="0.000003455444" iyz="0.000000074876" izz="0.000000165334"/>
-		</inertial>
-		<collision name="collision_base">
-			<origin xyz="-0.0025 0 -0.028" rpy="0 0 0"/>
-			<geometry>
-				<box size="0.005 0.015 0.075"/>
-			</geometry>
-		</collision>
-		<visual>
-			<origin xyz="0 0 0" rpy="0 0 0"/>
-			<geometry>
-				<mesh filename="package://dreamwalker_description/meshes/link_tibia1.stl" scale="0.001 0.001 0.001" />
+			<mass value="0.00730"/>
+			<origin xyz="-0.0025 0.0009 -0.032102" rpy="0 0 0"/>
+			<inertia ixx="0.0000050464" ixy="0" ixz="0" iyy="0.000004893134" iyz="0.00000009901" izz="0.00000018368"/>
+		</inertial>
+		<collision name="collision_base">
+			<origin xyz="-0.0025 0 -0.033" rpy="0 0 0"/>
+			<geometry>
+				<box size="0.005 0.015 0.085"/>
+			</geometry>
+		</collision>
+		<visual>
+			<origin xyz="0 0 0" rpy="0 0 0"/>
+			<geometry>
+				<mesh filename="package://dreamwalker_description/meshes/link_forearm1.stl" scale="0.001 0.001 0.001" />
 			</geometry>
 		</visual>
@@ -210,18 +211,18 @@
 	<link name="link_tibia2">
 		<inertial>
-			<mass value="0.00651"/>
-			<origin xyz="0.0025 0.000876 -0.027677" rpy="0 0 0"/>
-			<inertia ixx="0.000003593654" ixy="0" ixz="0" iyy="0.000003455444" iyz="0.000000074876" izz="0.000000165334"/>
-		</inertial>
-		<collision name="collision_base">
-			<origin xyz="0.0025 0 -0.028" rpy="0 0 0"/>
-			<geometry>
-				<box size="0.005 0.015 0.075"/>
-			</geometry>
-		</collision>
-		<visual>
-			<origin xyz="0 0 0" rpy="0 0 0"/>
-			<geometry>
-				<mesh filename="package://dreamwalker_description/meshes/link_tibia2.stl" scale="0.001 0.001 0.001" />
+			<mass value="0.00730"/>
+			<origin xyz="0.0025 0.0009 -0.032102" rpy="0 0 0"/>
+			<inertia ixx="0.0000050464" ixy="0" ixz="0" iyy="0.000004893134" iyz="0.00000009901" izz="0.00000018368"/>
+		</inertial>
+		<collision name="collision_base">
+			<origin xyz="0.0025 0 -0.033" rpy="0 0 0"/>
+			<geometry>
+				<box size="0.005 0.015 0.085"/>
+			</geometry>
+		</collision>
+		<visual>
+			<origin xyz="0 0 0" rpy="0 0 0"/>
+			<geometry>
+				<mesh filename="package://dreamwalker_description/meshes/link_forearm2.stl" scale="0.001 0.001 0.001" />
 			</geometry>
 		</visual>
@@ -229,18 +230,18 @@
 	<link name="link_tibia3">
 		<inertial>
-			<mass value="0.00651"/>
-			<origin xyz="-0.0025 -0.000876 -0.027677" rpy="0 0 0"/>
-			<inertia ixx="0.000003593654" ixy="0" ixz="0" iyy="0.000003455444" iyz="-0.000000074876" izz="0.000000165334"/>
-		</inertial>
-		<collision name="collision_base">
-			<origin xyz="-0.0025 0 -0.028" rpy="0 0 0"/>
-			<geometry>
-				<box size="0.005 0.015 0.075"/>
-			</geometry>
-		</collision>
-		<visual>
-			<origin xyz="0 0 0" rpy="0 0 0"/>
-			<geometry>
-				<mesh filename="package://dreamwalker_description/meshes/link_tibia3.stl" scale="0.001 0.001 0.001" />
+			<mass value="0.00730"/>
+			<origin xyz="-0.0025 0.0009 -0.032102" rpy="0 0 0"/>
+			<inertia ixx="0.0000050464" ixy="0" ixz="0" iyy="0.000004893134" iyz="0.00000009901" izz="0.00000018368"/>
+		</inertial>
+		<collision name="collision_base">
+			<origin xyz="-0.0025 0 -0.033" rpy="0 0 0"/>
+			<geometry>
+				<box size="0.005 0.015 0.085"/>
+			</geometry>
+		</collision>
+		<visual>
+			<origin xyz="0 0 0" rpy="0 0 0"/>
+			<geometry>
+				<mesh filename="package://dreamwalker_description/meshes/link_forearm1.stl" scale="0.001 0.001 0.001" />
 			</geometry>
 		</visual>
@@ -248,18 +249,18 @@
 	<link name="link_tibia4">
 		<inertial>
-			<mass value="0.00651"/>
-			<origin xyz="0.0025 -0.000876 -0.027677" rpy="0 0 0"/>
-			<inertia ixx="0.000003593654" ixy="0" ixz="0" iyy="0.000003455444" iyz="-0.000000074876" izz="0.000000165334"/>
-		</inertial>
-		<collision name="collision_base">
-			<origin xyz="0.0025 0 -0.028" rpy="0 0 0"/>
-			<geometry>
-				<box size="0.005 0.015 0.075"/>
-			</geometry>
-		</collision>
-		<visual>
-			<origin xyz="0 0 0" rpy="0 0 0"/>
-			<geometry>
-				<mesh filename="package://dreamwalker_description/meshes/link_tibia4.stl" scale="0.001 0.001 0.001" />
+			<mass value="0.00730"/>
+			<origin xyz="0.0025 0.0009 -0.032102" rpy="0 0 0"/>
+			<inertia ixx="0.0000050464" ixy="0" ixz="0" iyy="0.000004893134" iyz="0.00000009901" izz="0.00000018368"/>
+		</inertial>
+		<collision name="collision_base">
+			<origin xyz="0.0025 0 -0.033" rpy="0 0 0"/>
+			<geometry>
+				<box size="0.005 0.015 0.085"/>
+			</geometry>
+		</collision>
+		<visual>
+			<origin xyz="0 0 0" rpy="0 0 0"/>
+			<geometry>
+				<mesh filename="package://dreamwalker_description/meshes/link_forearm2.stl" scale="0.001 0.001 0.001" />
 			</geometry>
 		</visual>
@@ -271,15 +272,15 @@
 			<inertia ixx="0.000000043185" ixy="0" ixz="0" iyy="0.000000029326" iyz="-0.000000074876" izz="0.000000054089"/>
 		</inertial>
-		<collision name="collision_base">
-			<origin xyz="0 0 0" rpy="0 0 0"/>
-			<geometry>
-				<mesh filename="package://dreamwalker_description/meshes/link_foot.stl" scale="0.001 0.001 0.001" />
-			</geometry>
-			<contact_coefficient mu="100.0" mu2="100.0" k_p="10000.0"  k_d="100.0" />
-		</collision>
-		<visual>
-			<origin xyz="0 0 0" rpy="0 0 0"/>
-			<geometry>
-				<mesh filename="package://dreamwalker_description/meshes/link_foot.stl" scale="0.001 0.001 0.001" />
+		<collision>
+			<origin xyz="0 0 0" rpy="0 0 0"/>
+			<geometry>
+				<mesh filename="package://dreamwalker_description/meshes/link_foot.dae" scale="0.001 0.001 0.001" />
+			</geometry>
+			<!-- <contact_coefficient mu="100.0" mu2="100.0" k_p="10000.0"  k_d="100.0" /> -->
+		</collision>
+		<visual>
+			<origin xyz="0 0 0" rpy="0 0 0"/>
+			<geometry>
+				<mesh filename="package://dreamwalker_description/meshes/link_foot.dae" scale="0.001 0.001 0.001" />
 			</geometry>
 			<material name="black"/>
@@ -292,15 +293,15 @@
 			<inertia ixx="0.000000043185" ixy="0" ixz="0" iyy="0.000000029326" iyz="-0.000000074876" izz="0.000000054089"/>
 		</inertial>
-		<collision name="collision_base">
-			<origin xyz="0 0 0" rpy="0 0 0"/>
-			<geometry>
-				<mesh filename="package://dreamwalker_description/meshes/link_foot.stl" scale="0.001 0.001 0.001" />
-			</geometry>
-			<contact_coefficient mu="100.0" mu2="100.0" k_p="10000.0"  k_d="100.0" />
-		</collision>
-		<visual>
-			<origin xyz="0 0 0" rpy="0 0 0"/>
-			<geometry>
-				<mesh filename="package://dreamwalker_description/meshes/link_foot.stl" scale="0.001 0.001 0.001" />
+		<collision>
+			<origin xyz="0 0 0" rpy="0 0 0"/>
+			<geometry>
+				<mesh filename="package://dreamwalker_description/meshes/link_foot.dae" scale="0.001 0.001 0.001" />
+			</geometry>
+			<!-- <contact_coefficient mu="100.0" mu2="100.0" k_p="10000.0"  k_d="100.0" /> -->
+		</collision>
+		<visual>
+			<origin xyz="0 0 0" rpy="0 0 0"/>
+			<geometry>
+				<mesh filename="package://dreamwalker_description/meshes/link_foot.dae" scale="0.001 0.001 0.001" />
 			</geometry>
 			<material name="black"/>
@@ -313,15 +314,15 @@
 			<inertia ixx="0.000000043185" ixy="0" ixz="0" iyy="0.000000029326" iyz="-0.000000074876" izz="0.000000054089"/>
 		</inertial>
-		<collision name="collision_base">
-			<origin xyz="0 0 0" rpy="0 0 0"/>
-			<geometry>
-				<mesh filename="package://dreamwalker_description/meshes/link_foot.stl" scale="0.001 0.001 0.001" />
-			</geometry>
-			<contact_coefficient mu="100.0" mu2="100.0" k_p="10000.0"  k_d="100.0" />
-		</collision>
-		<visual>
-			<origin xyz="0 0 0" rpy="0 0 0"/>
-			<geometry>
-				<mesh filename="package://dreamwalker_description/meshes/link_foot.stl" scale="0.001 0.001 0.001" />
+		<collision>
+			<origin xyz="0 0 0" rpy="0 0 0"/>
+			<geometry>
+				<mesh filename="package://dreamwalker_description/meshes/link_foot.dae" scale="0.001 0.001 0.001" />
+			</geometry>
+			<!-- <contact_coefficient mu="100.0" mu2="100.0" k_p="10000.0"  k_d="100.0" /> -->
+		</collision>
+		<visual>
+			<origin xyz="0 0 0" rpy="0 0 0"/>
+			<geometry>
+				<mesh filename="package://dreamwalker_description/meshes/link_foot.dae" scale="0.001 0.001 0.001" />
 			</geometry>
 			<material name="black"/>
@@ -334,15 +335,15 @@
 			<inertia ixx="0.000000043185" ixy="0" ixz="0" iyy="0.000000029326" iyz="-0.000000074876" izz="0.000000054089"/>
 		</inertial>
-		<collision name="collision_base">
-			<origin xyz="0 0 0" rpy="0 0 0"/>
-			<geometry>
-				<mesh filename="package://dreamwalker_description/meshes/link_foot.stl" scale="0.001 0.001 0.001" />
-			</geometry>
-			<contact_coefficient mu="100.0" mu2="100.0" k_p="10000.0"  k_d="100.0" />
-		</collision>
-		<visual>
-			<origin xyz="0 0 0" rpy="0 0 0"/>
-			<geometry>
-				<mesh filename="package://dreamwalker_description/meshes/link_foot.stl" scale="0.001 0.001 0.001" />
+		<collision>
+			<origin xyz="0 0 0" rpy="0 0 0"/>
+			<geometry>
+				<mesh filename="package://dreamwalker_description/meshes/link_foot.dae" scale="0.001 0.001 0.001" />
+			</geometry>
+			<!-- <contact_coefficient mu="100.0" mu2="100.0" k_p="10000.0"  k_d="100.0" /> -->
+		</collision>
+		<visual>
+			<origin xyz="0 0 0" rpy="0 0 0"/>
+			<geometry>
+				<mesh filename="package://dreamwalker_description/meshes/link_foot.dae" scale="0.001 0.001 0.001" />
 			</geometry>
 			<material name="black"/>
@@ -435,5 +436,5 @@
 		<parent link="link_femur3"/>
 		<child link="link_tibia3"/>
-		<limit effort="30" velocity="1.0" lower="-2.09439" upper="0" />
+		<limit effort="30" velocity="1.0" lower="0" upper="2.09439" />
 		<!-- <dynamics damping="0.0" friction="1.0"/> -->
 	</joint>
@@ -443,33 +444,128 @@
 		<parent link="link_femur4"/>
 		<child link="link_tibia4"/>
-		<limit effort="30" velocity="1.0" lower="-2.09439" upper="0" />
+		<limit effort="30" velocity="1.0" lower="0" upper="2.09439" />
 		<!-- <dynamics damping="0.0" friction="1.0"/> -->
 	</joint>
 	<joint name="foot_joint1" type="fixed">
-		<origin xyz="-0.0025 0 -0.065" rpy="-0.52359 0 0"/>
+		<origin xyz="-0.0025 0 -0.075" rpy="-0.52359 0 0"/>
 		<parent link="link_tibia1"/>
 		<child link="link_foot1"/>
 	</joint>
 	<joint name="foot_joint2" type="fixed">
-		<origin xyz="0.0025 0 -0.065" rpy="-0.52359 0 0"/>
+		<origin xyz="0.0025 0 -0.075" rpy="-0.52359 0 0"/>
 		<parent link="link_tibia2"/>
 		<child link="link_foot2"/>
 	</joint>
 	<joint name="foot_joint3" type="fixed">
-		<origin xyz="-0.0025 0 -0.065" rpy="0.52359 0 0"/>
+		<origin xyz="-0.0025 0 -0.075" rpy="-0.52359 0 0"/>
 		<parent link="link_tibia3"/>
 		<child link="link_foot3"/>
 	</joint>
 	<joint name="foot_joint4" type="fixed">
-		<origin xyz="0.0025 0 -0.065" rpy="0.52359 0 0"/>
+		<origin xyz="0.0025 0 -0.075" rpy="-0.52359 0 0"/>
 		<parent link="link_tibia4"/>
 		<child link="link_foot4"/>
 	</joint>
-	<!-- ### GAZEBO ### -->
-	<gazebo>
-  		<plugin name="gazebo_ros_control" filename="libgazebo_ros_control.so">
-    		<robotNamespace>/dreamwalker</robotNamespace>
-  		</plugin>
-	</gazebo>
+	<!-- ### SENSORS ### -->
+	<link name="link_m_sensor">
+		<inertial>
+			<mass value="0.0102"/>
+			<origin xyz="0 0.01591 0.011" rpy="0 0 0"/>
+			<inertia ixx="0.000000566328" ixy="0" ixz="0" iyy="0.000002259218" iyz="-0.0000000944" izz="0.000002156532"/>
+		</inertial>
+		<collision name="collision_base">
+			<origin xyz="0 0.015 0.01125" rpy="0 0 0"/>
+			<geometry>
+				<box size="0.050 0.0293 0.0225"/>
+			</geometry>
+		</collision>
+		<visual>
+			<origin xyz="0 0 0" rpy="0 0 0"/>
+			<geometry>
+				<mesh filename="package://dreamwalker_description/meshes/link_fb_sensor.stl" scale="0.001 0.001 0.001" />
+			</geometry>
+		</visual>
+	</link>
+	<joint name="m_sensor_joint" type="revolute">
+		<origin xyz="0 0.095 0.005" rpy="0 0 0"/>
+		<parent link="main_body"/>
+		<child link="link_m_sensor"/>
+		<limit effort="1000" velocity="0.0" lower="0" upper="0" />
+	</joint>
+	<link name="link_b_sensor">
+		<inertial>
+			<mass value="0.0102"/>
+			<origin xyz="0 0.01591 0.011" rpy="0 0 0"/>
+			<inertia ixx="0.000000566328" ixy="0" ixz="0" iyy="0.000002259218" iyz="-0.0000000944" izz="0.000002156532"/>
+		</inertial>
+		<collision name="collision_base">
+			<origin xyz="0 0.015 0.01125" rpy="0 0 0"/>
+			<geometry>
+				<box size="0.050 0.0293 0.0225"/>
+			</geometry>
+		</collision>
+		<visual>
+			<origin xyz="0 0 0" rpy="0 0 0"/>
+			<geometry>
+				<mesh filename="package://dreamwalker_description/meshes/link_fb_sensor.stl" scale="0.001 0.001 0.001" />
+			</geometry>
+		</visual>
+	</link>
+	<joint name="b_sensor_joint" type="revolute">
+		<origin xyz="0 -0.095 0.005" rpy="0 0 3.141592"/>
+		<parent link="main_body"/>
+		<child link="link_b_sensor"/>
+		<limit effort="1000" velocity="0.0" lower="0" upper="0" />
+	</joint>
+	<link name="link_l_sensor">
+		<inertial>
+			<mass value="0.00983"/>
+			<origin xyz="0 0.01336 0.02495" rpy="0 0 0"/>
+			<inertia ixx="0.000002392374" ixy="0" ixz="0" iyy="0.000002455416" iyz="-0.000000093261" izz="0.000000406513"/>
+		</inertial>
+		<collision name="collision_base">
+			<origin xyz="0 0.015 0.025" rpy="0 0 0"/>
+			<geometry>
+				<box size="0.020 0.015 0.052"/>
+			</geometry>
+		</collision>
+		<visual>
+			<origin xyz="0 0 0" rpy="0 0 0"/>
+			<geometry>
+				<mesh filename="package://dreamwalker_description/meshes/link_rl_sensor.stl" scale="0.001 0.001 0.001" />
+			</geometry>
+		</visual>
+	</link>
+	<joint name="l_sensor_joint" type="revolute">
+		<origin xyz="-0.025 0.090 0.034" rpy="0 0 0.785398163"/>
+		<parent link="main_body"/>
+		<child link="link_l_sensor"/>
+		<limit effort="1000" velocity="0.0" lower="0" upper="0" />
+	</joint>
+	<link name="link_r_sensor">
+		<inertial>
+			<mass value="0.00983"/>
+			<origin xyz="0 0.01336 0.02495" rpy="0 0 0"/>
+			<inertia ixx="0.000002392374" ixy="0" ixz="0" iyy="0.000002455416" iyz="-0.000000093261" izz="0.000000406513"/>
+		</inertial>
+		<collision name="collision_base">
+			<origin xyz="0 0.015 0.025" rpy="0 0 0"/>
+			<geometry>
+				<box size="0.020 0.015 0.052"/>
+			</geometry>
+		</collision>
+		<visual>
+			<origin xyz="0 0 0" rpy="0 0 0"/>
+			<geometry>
+				<mesh filename="package://dreamwalker_description/meshes/link_rl_sensor.stl" scale="0.001 0.001 0.001" />
+			</geometry>
+		</visual>
+	</link>
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
Commit message: robot can jump

File: dreamwalker_description/urdf/dreamwalker_dummy.xacro (robot description, xacro)
@@ -382,5 +382,5 @@
 		<parent link="main_body"/>
 		<child link="link_shoulder1"/>
-		<limit effort="30" velocity="5.0" lower="-0.5235987755983" upper="0.5235987755983" />
+		<limit effort="2.5" velocity="1.0" lower="-0.5235987755983" upper="0.5235987755983" />
 		<!-- <dynamics damping="0.0" friction="1.0"/> -->
 	</joint>
@@ -390,5 +390,5 @@
 		<parent link="main_body"/>
 		<child link="link_shoulder2"/>
-		<limit effort="30" velocity="5.0" lower="-0.5235987755983" upper="0.5235987755983" />
+		<limit effort="2.5" velocity="1.0" lower="-0.5235987755983" upper="0.5235987755983" />
 		<!-- <dynamics damping="0.0" friction="1.0"/> -->
 	</joint>
@@ -398,5 +398,5 @@
 		<parent link="main_body"/>
 		<child link="link_shoulder3"/>
-		<limit effort="30" velocity="5.0" lower="-0.5235987755983" upper="0.5235987755983" />
+		<limit effort="2.5" velocity="1.0" lower="-0.5235987755983" upper="0.5235987755983" />
 		<!--<dynamics damping="0.0" friction="1.0"/> -->
 	</joint>
@@ -406,5 +406,5 @@
 		<parent link="main_body"/>
 		<child link="link_shoulder4"/>
-		<limit effort="30" velocity="1.0" lower="-0.52359" upper="0.52359" />
+		<limit effort="2.5" velocity="1.0" lower="-0.52359" upper="0.52359" />
 		<!--<dynamics damping="0.0" friction="1.0"/> -->
 	</joint>
@@ -414,5 +414,5 @@
 		<parent link="link_shoulder1"/>
 		<child link="link_femur1"/>
-		<limit effort="30" velocity="1.0" lower="-1.57079" upper="1.57079" />
+		<limit effort="2.5" velocity="1.0" lower="-1.57079" upper="1.57079" />
 		<!-- <dynamics damping="0.0" friction="1.0"/> -->
 	</joint>
@@ -422,5 +422,5 @@
 		<parent link="link_shoulder2"/>
 		<child link="link_femur2"/>
-		<limit effort="30" velocity="1.0" lower="-1.57079" upper="1.57079" />
+		<limit effort="2.5" velocity="1.0" lower="-1.57079" upper="1.57079" />
 		<!-- <dynamics damping="0.0" friction="1.0"/> -->
 	</joint>
@@ -430,5 +430,5 @@
 		<parent link="link_shoulder3"/>
 		<child link="link_femur3"/>
-		<limit effort="30" velocity="1.0" lower="-1.57079" upper="1.57079" />
+		<limit effort="2.5" velocity="1.0" lower="-1.57079" upper="1.57079" />
 		<!-- <dynamics damping="0.0" friction="1.0"/> -->
 	</joint>
@@ -438,5 +438,5 @@
 		<parent link="link_shoulder4"/>
 		<child link="link_femur4"/>
-		<limit effort="30" velocity="1.0" lower="-1.57079" upper="1.57079" />
+		<limit effort="2.5" velocity="1.0" lower="-1.57079" upper="1.57079" />
 		<!-- <dynamics damping="0.0" friction="1.0"/> -->
 	</joint>
@@ -446,5 +446,5 @@
 		<parent link="link_femur1"/>
 		<child link="link_tibia1"/>
-		<limit effort="30" velocity="1.0" lower="0" upper="2.09439" />
+		<limit effort="2.5" velocity="1.0" lower="0" upper="2.09439" />
 		<!-- <dynamics damping="0.0" friction="1.0"/> -->
 	</joint>
@@ -454,5 +454,5 @@
 		<parent link="link_femur2"/>
 		<child link="link_tibia2"/>
-		<limit effort="30" velocity="1.0" lower="0" upper="2.09439" />
+		<limit effort="2.5" velocity="1.0" lower="0" upper="2.09439" />
 		<!-- <dynamics damping="0.0" friction="1.0"/> -->
 	</joint>
@@ -462,5 +462,5 @@
 		<parent link="link_femur3"/>
 		<child link="link_tibia3"/>
-		<limit effort="30" velocity="1.0" lower="0" upper="2.09439" />
+		<limit effort="2.5" velocity="1.0" lower="0" upper="2.09439" />
 		<!-- <dynamics damping="0.0" friction="1.0"/> -->
 	</joint>
@@ -470,5 +470,5 @@
 		<parent link="link_femur4"/>
 		<child link="link_tibia4"/>
-		<limit effort="30" velocity="1.0" lower="0" upper="2.09439" />
+		<limit effort="2.5" velocity="1.0" lower="0" upper="2.09439" />
 		<!-- <dynamics damping="0.0" friction="1.0"/> -->
 	</joint>

Commit message: main.py let's to control robot as desired

File: dreamwalker_description/urdf/dreamwalker_dummy.xacro (robot description, xacro)
@@ -446,5 +446,5 @@
 		<parent link="link_femur1"/>
 		<child link="link_tibia1"/>
-		<limit effort="2.5" velocity="1.0" lower="0" upper="2.09439" />
+		<limit effort="2.5" velocity="1.0" lower="0" upper="2.617993878" />
 		<!-- <dynamics damping="0.0" friction="1.0"/> -->
 	</joint>
@@ -454,5 +454,5 @@
 		<parent link="link_femur2"/>
 		<child link="link_tibia2"/>
-		<limit effort="2.5" velocity="1.0" lower="0" upper="2.09439" />
+		<limit effort="2.5" velocity="1.0" lower="0" upper="2.617993878" />
 		<!-- <dynamics damping="0.0" friction="1.0"/> -->
 	</joint>
@@ -462,5 +462,5 @@
 		<parent link="link_femur3"/>
 		<child link="link_tibia3"/>
-		<limit effort="2.5" velocity="1.0" lower="0" upper="2.09439" />
+		<limit effort="2.5" velocity="1.0" lower="0" upper="2.617993878" />
 		<!-- <dynamics damping="0.0" friction="1.0"/> -->
 	</joint>
@@ -470,5 +470,5 @@
 		<parent link="link_femur4"/>
 		<child link="link_tibia4"/>
-		<limit effort="2.5" velocity="1.0" lower="0" upper="2.09439" />
+		<limit effort="2.5" velocity="1.0" lower="0" upper="2.617993878" />
 		<!-- <dynamics damping="0.0" friction="1.0"/> -->
 	</joint>

File: dreamwalker_description/urdf/dreamwalker_test.xacro (robot description, xacro)
@@ -420,5 +420,5 @@
 		<parent link="link_femur1"/>
 		<child link="link_tibia1"/>
-		<limit effort="2.5" velocity="1.0" lower="0" upper="2.09439" />
+		<limit effort="2.5" velocity="1.0" lower="0" upper="2.617993878" />
 		<!-- <dynamics damping="0.0" friction="1.0"/> -->
 	</joint>
@@ -428,5 +428,5 @@
 		<parent link="link_femur2"/>
 		<child link="link_tibia2"/>
-		<limit effort="2.5" velocity="1.0" lower="0" upper="2.09439" />
+		<limit effort="2.5" velocity="1.0" lower="0" upper="2.617993878" />
 		<!-- <dynamics damping="0.0" friction="1.0"/> -->
 	</joint>
@@ -436,5 +436,5 @@
 		<parent link="link_femur3"/>
 		<child link="link_tibia3"/>
-		<limit effort="2.5" velocity="1.0" lower="0" upper="2.09439" />
+		<limit effort="2.5" velocity="1.0" lower="0" upper="2.617993878" />
 		<!-- <dynamics damping="0.0" friction="1.0"/> -->
 	</joint>
@@ -444,5 +444,5 @@
 		<parent link="link_femur4"/>
 		<child link="link_tibia4"/>
-		<limit effort="2.5" velocity="1.0" lower="0" upper="2.09439" />
+		<limit effort="2.5" velocity="1.0" lower="0" upper="2.617993878" />
 		<!-- <dynamics damping="0.0" friction="1.0"/> -->
 	</joint>
